Commit message: i can fly on KMHE finally

File: quads/clara/clara.xacro (robot description, xacro)
@@ -19,4 +19,6 @@
   <xacro:property name="moment_constant" value="0.022" /> <!-- [Nm/N] 0.016 ct -->
   <xacro:property name="max_thrust" value="8.7" /> <!-- [N] Max thrust of individual rotor-->
+  <xacro:property name="max_input_value" value="1.0" /> <!-- # Motors at full thrust -->
+  <xacro:property name="min_input_value" value="0.0" /> <!-- # Motors turned off -->
   <xacro:property name="time_constant_up" value="0.033" /> <!-- [s] -->
   <xacro:property name="time_constant_down" value="0.033" /> <!-- [s] -->

File: quads/clark/clark.xacro (robot description, xacro)
@@ -19,4 +19,6 @@
   <xacro:property name="moment_constant" value="0.022" /> <!-- [Nm/N] 0.016 ct -->
   <xacro:property name="max_thrust" value="15.75" /> <!-- [N] Max thrust of individual rotor-->
+  <xacro:property name="max_input_value" value="0.5" /> <!-- # Motors at full thrust -->
+  <xacro:property name="min_input_value" value="0" /> <!-- # Motors turned off -->
   <xacro:property name="time_constant_up" value="0.033" /> <!-- [s] -->
   <xacro:property name="time_constant_down" value="0.033" /> <!-- [s] -->

Commit message: KMHE and DMHE both work and quad is able to fly using state estimations

File: quads/clara/clara.xacro (robot description, xacro)
@@ -18,5 +18,5 @@
   <xacro:property name="motor_constant" value="1.56252e-06" /> <!-- [kg m/s^2] kf-->
   <xacro:property name="moment_constant" value="0.022" /> <!-- [Nm/N] 0.016 ct -->
-  <xacro:property name="max_thrust" value="8.7" /> <!-- [N] Max thrust of individual rotor-->
+  <xacro:property name="max_thrust" value="8.35" /> <!-- [N] Max thrust of individual rotor-->
   <xacro:property name="max_input_value" value="1.0" /> <!-- # Motors at full thrust -->
   <xacro:property name="min_input_value" value="0.0" /> <!-- # Motors turned off -->
